File: spinner.kicad_pcb (KiCad board)
At the start: 2 copper layers, 147 x 147 mm, 113 parts, among them J1 Micro_SD_Card, SW1 SW_SPDT, U1 AP63205WU, U2 RS0102, U3 SFH617A-3X006, U4 SFH617A-3X006, U5 SFH617A-3X006, U6 ESP32-S3-WROOM-1

Commit message: Layout things.
Parts:
- removed H4, H5, H6, H7, H8, H9: MountingHole, MountingHole:MountingHole_3mm
- moved H1 130.0 mm to (158.7, 105.0)
- moved H2 120.8 mm to (141.3, 105.0)
- moved H3 112.4 mm to (150.0, 90.0)
- moved U5 65.1 mm to (206.3, 132.5)
- moved U3 0.57 mm to (215.0, 100.6), turned to 179.5 degrees
