File: spinner.kicad_pcb (KiCad board)
At the start: 2 copper layers, 147 x 147 mm, 134 parts, among them J1 Micro_SD_Card, J301 USB_C_Receptacle_USB2.0_16P, SW1 SW_SPDT, SW301 RESET, SW302 BOOT, U2 RS0102, U301 BQ24073RGT, U302 SPX3819M5-L-3-3, U303 TPS61022, u10 ESP32-S3-WROOM-1

Commit message: Some board layout.
Parts:
- moved R308 0.74 mm to (199.6, 122.2)
- moved TP1 0.74 mm to (162.4, 30.3)
- moved R307 0.74 mm to (207.2, 76.6)
- moved D325 0.74 mm to (206.2, 85.3)
- moved D328 0.74 mm to (95.2, 101.3)
- moved L2 0.74 mm to (188.1, 118.2)
- moved R309 0.74 mm to (199.6, 119.2)
- moved BT3 0.74 mm to (172.7, 112.3)
- moved D202 0.74 mm to (145.0, 96.3)
- moved D203 0.74 mm to (142.4, 94.8)
- moved D207 0.74 mm to (132.0, 88.8)
- moved D216 0.74 mm to (108.6, 75.3)
- moved D221 0.74 mm to (95.6, 67.8)
- moved D222 0.74 mm to (93.0, 66.3)
- moved D307 0.74 mm to (168.4, 88.8)
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Routing:
- net Net-(JP301-C): track 0.00 -> 9.65 mm
- net GND: track 0.00 -> 7.46 mm, vias 0 -> 5
- net Net-(U303-FB): track 0.00 -> 7.32 mm
- net /dat_2: track 0.00 -> 5.70 mm
- net /dat_3: track 0.00 -> 5.32 mm
- net /dat_0: track 0.00 -> 5.12 mm
- net /spi_clk: track 0.00 -> 5.03 mm
- net /cmd: track 0.00 -> 4.95 mm
- net /dat_1: track 0.00 -> 4.81 mm
- net Net-(U303-SW): track 0.00 -> 1.52 mm
- net Net-(D321-CO): track 0.00 -> 1.41 mm
- net Net-(D321-DO): track 0.00 -> 1.41 mm
- net Net-(D101-DO): track 0.00 -> 1.40 mm
- net Net-(D101-CO): track 0.00 -> 1.40 mm
- net Net-(D316-DO): track 0.00 -> 1.40 mm
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- added copper zone on F.Cu, net BATT_COND
- added copper zone on F.Cu, net GND
- added copper zone on F.Cu, net Net-(U303-SW)
