File: spinner.kicad_sch (KiCad schematic)
At the start: 141 parts, among them J1 Micro_SD_Card, J301 USB_C_Receptacle_USB2.0_16P, J303 Conn_01x03_Pin, SW1 SW_SPDT, SW301 RESET, SW302 BOOT, U2 RS0102, U301 BQ24073RGT, U302 SPX3819M5-L-3-3, U303 TPS61022, u10 ESP32-S3-WROOM-1

Commit message: Changed the power plane to 3.3v from 5v.
Made footprint for battery jumper.
Did more routing.
Parts:
- J303: footprint Connector_PinHeader_1.00mm:PinHeader_1x03_P1.00mm_Vertical -> Library:PinHeader_1x03_P2.54mm_HRZ_SMD_Pin1Left
- renumbered D101 to D100, D0 to D101
Connections:
- net CI: now also D100.2 (CI); no longer D101.2 (CI)
- net DI: now also D100.1 (DI); no longer D101.1 (DI)
- net at D102.1 (DI): now also D101.6 (DO); no longer D100.6 (DO)
- net at D102.2 (CI): now also D101.5 (CO); no longer D100.5 (CO)
- new net: D100.6 (DO), D101.1 (DI)
- new net: D100.5 (CO), D101.2 (CI)
Other:
- moved on the sheet: D100, D101
